Commit message: first config works

File: alpha_img_description/urdf/base.urdf.xacro (robot description, xacro)
@@ -3,5 +3,5 @@
     <link name="nose_tip_link">
         <visual>
-            <origin xyz="00.0 0.0 0.0" rpy="0.0 0.0 0.0"/>
+            <origin xyz="0.0 0.0 0.0" rpy="0.0 0.0 0.0"/>
             <geometry>
                 <mesh filename="package://alpha_img_description/mesh/alpha_img_rviz.stl" scale="0.001 0.001 0.001"/>
@@ -11,5 +11,5 @@
     <link name="base_link"/>
     <joint name="base_link" type="fixed">
-        <origin xyz="0.72 0.0 0.0" rpy="0.0 0.0 0.0"/>
+        <origin xyz="0.70 0.0 0.0" rpy="0.0 0.0 0.0"/>
         <parent link="base_link"/>
         <child link="nose_tip_link"/>
@@ -23,75 +23,74 @@
     <link name="imu"/>
     <joint name="imu_joint" type="fixed">
-        <origin xyz="-0.2 -0.07 0.0" rpy="3.1415926 0.0 0.0"/>
-        <parent link="base_link"/>
+        <origin xyz="-0.6867 -0.0625 -0.0381" rpy="3.1415926 0.0 0.0"/>
+        <parent link="nose_tip_link"/>
         <child link="imu"/>
     </joint>
     <link name="imu_sf"/>
-    <joint name="imu__sf_joint" type="fixed">
-        <origin xyz="0.0 0.0 0.0" rpy="0.0 0.0 0.0"/>
-        <parent link="imu"/>
+    <joint name="imu_sf_joint" type="fixed">
+        <origin xyz="-0.6867 -0.0625 -0.0381" rpy="3.1415926 0.0 0.0"/>
+        <parent link="nose_tip_link"/>
         <child link="imu_sf"/>
     </joint>
     <link name="dvl"/>
     <joint name="dvl_joint" type="fixed">
-        <origin xyz="0.51 0.0 -0.1" rpy="3.1415926 0.0 0.0"/>
-        <parent link="base_link"/>
+        <origin xyz="-1.005 0.0 -0.1" rpy="3.1415926 0.0 0.0"/>
+        <parent link="nose_tip_link"/>
         <child link="dvl"/>
     </joint>
      <link name="dvl_sf"/>
     <joint name="dvl_sf_joint" type="fixed">
-        <origin xyz="0.51 0.0 -0.1" rpy="0.0 0.0 0.0"/>
-        <parent link="base_link"/>
+        <origin xyz="-1.005 0.0 -0.1" rpy="0.0 0.0 0.0"/>
+        <parent link="nose_tip_link"/>
         <child link="dvl_sf"/>
     </joint>
     <link name="gps"/>
     <joint name="gps_joint" type="fixed">
-        <origin xyz="0.05 0.0 0.32" rpy="3.1415926 0.0 0.0"/>
-        <parent link="base_link"/>
+        <origin xyz="-0.7 0.0 0.3" rpy="3.1415926 0.0 0.0"/>
+        <parent link="nose_tip_link"/>
         <child link="gps"/>
     </joint>
     <link name="pressure"/>
     <joint name="pressure_joint" type="fixed">
-        <origin xyz="0.3 0.0 0.05" rpy="3.1415926 0.0 0.0"/>
-        <parent link="base_link"/>
+        <origin xyz="-0.4073 -0.0625 0.0" rpy="3.1415926 0.0 0.0"/>
+        <parent link="nose_tip_link"/>
         <child link="pressure"/>
     </joint>
     <link name="ping360_link"/>
     <joint name="ping360_joint" type="fixed">
-        <origin xyz="0.63 0.0 -0.085" rpy="0.0 0.0 3.1415926"/>
-        <parent link="base_link"/>
+        <origin xyz="-0.01 0.12192 0.0" rpy="-1.57079632679 0.0 3.1415926"/>
+        <parent link="nose_tip_link"/>
         <child link="ping360_link"/>
+    </joint>
+    <link name="oculus"/>
+    <joint name="fls_joint" type="fixed">
+        <origin xyz="0.0 -0.04 -0.09" rpy="3.1415926 0.436332306 0.0"/>
+        <parent link="nose_tip_link"/>
+        <child link="oculus"/>
     </joint>
     <!-- thrusters -->
     <link name="surge_thruster_link"/>
     <joint name="surge_thruster_joint" type="fixed">
-        <origin xyz="-0.77 0.0 0.0" rpy="0.0 0.0 0.0"/>
-        <parent link="base_link"/>
+        <origin xyz="-1.4 0.0 0.0" rpy="0.0 0.0 0.0"/>
+        <parent link="nose_tip_link"/>
         <child link="surge_thruster_link"/>
     </joint>
     <link name="heave_bow_thruster_link"/>
     <joint name="heave_bow_thruster_joint" type="fixed">
-        <origin xyz="0.387 0.0 0.0" rpy="0.0 -1.57079632679 0.0"/>
-        <parent link="base_link"/>
+        <origin xyz="-0.2295 0.0 0.0" rpy="0.0 -1.57079632679 0.0"/>
+        <parent link="nose_tip_link"/>
         <child link="heave_bow_thruster_link"/>
     </joint>
     <link name="heave_stern_thruster_link"/>
     <joint name="heave_stern_thruster_joint" type="fixed">
-        <origin xyz="-0.4 0.0 0.0" rpy="0.0 -1.57079632679 0.0"/>
-        <parent link="base_link"/>
+        <origin xyz="-0.88 0.0 0.0" rpy="0.0 -1.57079632679 0.0"/>
+        <parent link="nose_tip_link"/>
         <child link="heave_stern_thruster_link"/>
     </joint>
     <link name="sway_bow_thruster_link"/>
     <joint name="sway_bow_thruster_joint" type="fixed">
-        <origin xyz="0.51 0.0 0.0" rpy="0.0 0.0 1.57079632679"/>
-        <parent link="base_link"/>
+        <origin xyz="-1.005 0.0 0.0" rpy="0.0 0.0 1.57079632679"/>
+        <parent link="nose_tip_link"/>
         <child link="sway_bow_thruster_link"/>
     </joint>
-    <!-- perception sensors -->
-    <!-- <link name="mss"/>
-    <joint name="mss_joint" type="fixed">
-        <origin xyz="0.65 0.0 0.0" rpy="3.1415926 1.5707963 0.0"/>
-        <parent link="base_link"/>
-        <child link="mss"/>
-    </joint> -->
 </robot>

Commit message: change the tf & launchs

File: alpha_img_description/urdf/base.urdf.xacro (robot description, xacro)
@@ -11,5 +11,5 @@
     <link name="base_link"/>
     <joint name="base_link" type="fixed">
-        <origin xyz="0.70 0.0 0.0" rpy="0.0 0.0 0.0"/>
+        <origin xyz="0.825 0.0 0.0" rpy="0.0 0.0 0.0"/>
         <parent link="base_link"/>
         <child link="nose_tip_link"/>
@@ -23,5 +23,5 @@
     <link name="imu"/>
     <joint name="imu_joint" type="fixed">
-        <origin xyz="-0.6867 -0.0625 -0.0381" rpy="3.1415926 0.0 0.0"/>
+        <origin xyz="-0.8117 -0.0625 -0.0381" rpy="3.1415926 0.0 0.0"/>
         <parent link="nose_tip_link"/>
         <child link="imu"/>
@@ -35,5 +35,5 @@
     <link name="dvl"/>
     <joint name="dvl_joint" type="fixed">
-        <origin xyz="-1.005 0.0 -0.1" rpy="3.1415926 0.0 0.0"/>
+        <origin xyz="-1.13 0.0 -0.14" rpy="3.1415926 0.0 3.1415926"/>
         <parent link="nose_tip_link"/>
         <child link="dvl"/>
@@ -47,5 +47,5 @@
     <link name="gps"/>
     <joint name="gps_joint" type="fixed">
-        <origin xyz="-0.7 0.0 0.3" rpy="3.1415926 0.0 0.0"/>
+        <origin xyz="-0.51 0.0 0.395" rpy="3.1415926 0.0 0.0"/>
         <parent link="nose_tip_link"/>
         <child link="gps"/>
@@ -53,5 +53,5 @@
     <link name="pressure"/>
     <joint name="pressure_joint" type="fixed">
-        <origin xyz="-0.4073 -0.0625 0.0" rpy="3.1415926 0.0 0.0"/>
+        <origin xyz="-0.508 -0.0625 0.0" rpy="3.1415926 0.0 0.0"/>
         <parent link="nose_tip_link"/>
         <child link="pressure"/>
@@ -59,5 +59,5 @@
     <link name="ping360_link"/>
     <joint name="ping360_joint" type="fixed">
-        <origin xyz="-0.01 0.12192 0.0" rpy="-1.57079632679 0.0 3.1415926"/>
+        <origin xyz="-0.1 0.12192 0.0" rpy="-1.57079632679 0.0 3.1415926"/>
         <parent link="nose_tip_link"/>
         <child link="ping360_link"/>
@@ -65,5 +65,5 @@
     <link name="oculus"/>
     <joint name="fls_joint" type="fixed">
-        <origin xyz="0.0 -0.04 -0.09" rpy="3.1415926 0.436332306 0.0"/>
+        <origin xyz="0.0 -0.04 -0.09" rpy="3.1415926 0.261799383 0.0"/>
         <parent link="nose_tip_link"/>
         <child link="oculus"/>
@@ -72,5 +72,5 @@
     <link name="surge_thruster_link"/>
     <joint name="surge_thruster_joint" type="fixed">
-        <origin xyz="-1.4 0.0 0.0" rpy="0.0 0.0 0.0"/>
+        <origin xyz="-1.525 0.0 0.0" rpy="0.0 0.0 0.0"/>
         <parent link="nose_tip_link"/>
         <child link="surge_thruster_link"/>
@@ -78,5 +78,5 @@
     <link name="heave_bow_thruster_link"/>
     <joint name="heave_bow_thruster_joint" type="fixed">
-        <origin xyz="-0.2295 0.0 0.0" rpy="0.0 -1.57079632679 0.0"/>
+        <origin xyz="-0.3545 0.0 0.0" rpy="0.0 -1.57079632679 0.0"/>
         <parent link="nose_tip_link"/>
         <child link="heave_bow_thruster_link"/>
@@ -84,5 +84,5 @@
     <link name="heave_stern_thruster_link"/>
     <joint name="heave_stern_thruster_joint" type="fixed">
-        <origin xyz="-0.88 0.0 0.0" rpy="0.0 -1.57079632679 0.0"/>
+        <origin xyz="-1.005 0.0 0.0" rpy="0.0 -1.57079632679 0.0"/>
         <parent link="nose_tip_link"/>
         <child link="heave_stern_thruster_link"/>
@@ -90,5 +90,5 @@
     <link name="sway_bow_thruster_link"/>
     <joint name="sway_bow_thruster_joint" type="fixed">
-        <origin xyz="-1.005 0.0 0.0" rpy="0.0 0.0 1.57079632679"/>
+        <origin xyz="-1.130 0.0 0.0" rpy="0.0 0.0 1.57079632679"/>
         <parent link="nose_tip_link"/>
         <child link="sway_bow_thruster_link"/>

Commit message: update changes after allen harbor test

File: alpha_img_description/urdf/base.urdf.xacro (robot description, xacro)
@@ -88,9 +88,9 @@
         <child link="heave_stern_thruster_link"/>
     </joint>
-    <link name="sway_bow_thruster_link"/>
-    <joint name="sway_bow_thruster_joint" type="fixed">
+    <link name="sway_stern_thruster_link"/>
+    <joint name="sway_stern_thruster_joint" type="fixed">
         <origin xyz="-1.130 0.0 0.0" rpy="0.0 0.0 1.57079632679"/>
         <parent link="nose_tip_link"/>
-        <child link="sway_bow_thruster_link"/>
+        <child link="sway_stern_thruster_link"/>
     </joint>
 </robot>

Commit message: config after allen harbor test at 7_26_2024

File: alpha_img_description/urdf/base.urdf.xacro (robot description, xacro)
@@ -23,5 +23,6 @@
     <link name="imu"/>
     <joint name="imu_joint" type="fixed">
-        <origin xyz="-0.8117 -0.0625 -0.0381" rpy="3.1415926 0.0 0.0"/>
+        <!-- <origin xyz="-0.8117 -0.0625 -0.0381" rpy="3.1415926 0.0 0.0"/> -->
+        <origin xyz="-0.8117 -0.0625 -0.0381" rpy="0.0 0.0 0.0"/>
         <parent link="nose_tip_link"/>
         <child link="imu"/>
